File: kicad/arduino-blue-pill-scope-perfboard.kicad_pcb (KiCad board)
At the start: 4 copper layers, 53.3 x 66 mm, 26 parts, among them J1 Header_1x6_male, J2 Header_1x1_male, J3 Header_1x1_male, J6 Header_1x1_male, U2 LM358, U3 BluePill_STM32F103C8T6

Commit message: Updated kicad project
Parts:
- added C11: 10u, dvhx-kicad-library-2:C_0805, B.Cu at (161.8, 45.7)
- added C12: 10u, dvhx-kicad-library-2:C_0805, B.Cu at (161.8, 53.6)
- added U1: ME6209A30, dvhx-kicad-library-2:SOT23-GOI, B.Cu at (161.3, 48.8)
- R2: value 2M2 -> 1M
Connections:
- D3 pad K: 5V -> 3V3
- D6 pad K: 5V -> 3V3
- R2 pad 2: 5V -> 3V3
- R6 pad 2: 5V -> 3V3
Routing:
- net GND: track 175.8 -> 195.8 mm
- net 3V3: track 41.5 -> 59.9 mm
- net 5V: track 114.0 -> 110.2 mm, vias 0 -> 2
- net 3V0: track 0.00 -> 3.68 mm
