File: kicad/arduino-blue-pill-scope-perfboard.kicad_sch (KiCad schematic)
At the start: 51 parts, among them J1 Header_1x6_male, J2 Header_1x1_male, J3 Header_1x1_male, J4 Header_1x1_male, J5 Header_1x1_male, J6 Header_1x1_male, U2 LM358, U3 BluePill_STM32F103C8T6, U4 LM358

Commit message: Updated kicad project
Parts:
- added C11, C12: 10u, dvhx-kicad-library-2:C_0805, symbol dvhx-kicad-library-2:C
- added U1: ME6209A30, dvhx-kicad-library-2:SOT23-GOI, symbol dvhx-kicad-library-2:ME6209A30
- R2: value 2M2 -> 1M
Connections:
- net 3V3: now also D11.K, D3.K, D6.K, D9.K, R11.2, R13.2, R2.2, R6.2
- net 5V: now also C11.1, U1.I; no longer D11.K, D3.K, D6.K, D9.K, R11.2, R13.2, R2.2, R6.2
- net GND: now also C11.2, C12.2, U1.G
- new net 3V0: C12.1, U1.O
Other:
- note added: "(this range was not tested)"
- note added: "*rev2"
- note added: "Not needed, use 3v3 out of blue pill"
